File: hardware/shield.sch (EAGLE design)
At the start: 16 parts

Commit message: mroe drones
Parts:
- added BAT: (no value), SparkFun-Connectors:M022.54MM_SCREWTERM
- added C10, C12, C8: 0.1uF, rcl:C-EUC1206
- added C11: 10uF, rcl:CPOL-EU153CLV-0405
- added C6: 100uF, rcl:CPOL-EU153CLV-0605
- added C7, C9: 1000uF, rcl:CPOL-EU153CLV-1012
- added D1: 1N5822, diode:DIODE-DO-214AC
- added IC2: AMS1117-3.3, v-reg:LD117AS12TR
- added IC3: 24C32ASN, microchip:24C32ASN
- added J$1: SMA_EDGE, SparkFun-Connectors:SMA_EDGE
- added JP1: (no value), jumper:JP1E
- added L1: SRR1210, inductor-bourns:SRR1210
- added L2: (no value), rcl:L-EUL2012C
- added LED1: (no value), led:LEDSMT1206
- added Q1: MOSFET-PCHANNEL_SOT23-3, Simplex-DiscreteSemi:MOSFET-PCHANNEL_SOT23-3
- added R10, R9: 4k7, resistor:R-EU_R1206
- added R11, R6, R7: 1k, resistor:R-EU_R1206
- added R12, R13: 3.9k, resistor:R-EU_R1206
- added R8: 22R, resistor:R-EU_R1206
- added SV1: (no value), con-lstb:MA04-2
- added SV10: DISTANCE, con-lstb:MA03-1
- added SV2: MOTOR0, con-lstb:MA03-1
- added SV3: MOTOR1, con-lstb:MA03-1
- added SV4: MOTOR2, con-lstb:MA03-1
- added SV5: MOTOR3, con-lstb:MA03-1
- added SV6: MOTOR4, con-lstb:MA03-1
- added SV7: MOTOR5, con-lstb:MA03-1
- added SV8: MOTOR6, con-lstb:MA03-1
- added SV9: MOTOR7, con-lstb:MA03-1
- added U$2: DMMT5401, Erle:DMMT5401
- added U$6: BLOX-NEO-6M, microduino:BLOX-NEO-6M
- U$1: value MCP3008SL -> ADS1015IDGT; device MCP3008:MCP3008SL -> bt_adc:ADS1015IDGT
Connections:
- removed net RPI1: RPI.1
- removed net RPI9: RPI.9
- new net +5V: C7.+, IC1.FBACK, IC2.IN, L1.2, Q1.D, SV10.2, U$2.6
- new net N$10: LED1.C, U$6.TIMEPULSE
- new net N$11: R7.1, U$6.MOSI/CFG_COM0
- new net N$12: SV1.3
- new net N$13: R8.2, U$6.RESERVED2, U$6.VCC_RF
- new net N$14: L2.2, R8.1
- new net N$15: J$1.SIGNAL, L2.1, U$6.RF_IN
- new net N$16: R9.2, U$2.1, U$2.2, U$2.3
- new net N$17: Q1.G, R10.2, U$2.4
- new net N$18: SV1.8
- new net N$21: IC3.WP, JP1.2, R11.1
- new net N$5: SV10.3, U$1.AIN1
- new net N$6: U$1.AIN2
- new net N$7: D1.A, IC1.VO, L1.1
- new net N$8: LED1.A, R6.2
- new net N$9: U$1.ALERT
- new net PWM0: PWM.PWM0, SV2.1
- new net PWM1: PWM.PWM1, SV3.1
- new net PWM10: PWM.PWM10
- new net PWM11: PWM.PWM11
- new net PWM12: PWM.PWM12
- new net PWM13: PWM.PWM13
- new net PWM14: PWM.PWM14
- new net PWM15: PWM.PWM15
- new net PWM2: PWM.PWM2, SV4.1
- new net PWM3: PWM.PWM3, SV5.1
- new net PWM4: PWM.PWM4, SV6.1
- new net PWM5: PWM.PWM5, SV7.1
- new net PWM6: PWM.PWM6, SV8.1
- new net PWM7: PWM.PWM7, SV9.1
- new net PWM8: PWM.PWM8
- new net PWM9: PWM.PWM9
- new net RPI27: IC3.SDA, R12.2
- new net RPI28: IC3.SCL, R13.1
- net +12V: now also BAT.2, C6.+
- net +3V3: now also C10.2, C11.+, C12.1, C8.1, C9.+, IC2.OUT, IC3.VCC, R11.2, R12.1, R13.2, R6.1, SV1.2, SV2.2, SV3.2, SV4.2, SV5.2, SV6.2, SV7.2, SV8.2, SV9.2, U$6.VCC; no longer U$1.VREF
- net GND: now also BAT.1, C10.1, C11.-, C12.2, C6.-, C7.-, C8.2, C9.-, D1.C, IC1.!EN, IC1.GND, IC2.ADJ, IC3.A0, IC3.A1, IC3.A2, IC3.GND, IMU.ADO/SDO, IMU.FSYNC, J$1.GND@0, J$1.GND@1, J$1.GND@2, J$1.GND@3, JP1.1, R10.1, R7.2, R9.1, RPI.14, RPI.20, RPI.25, RPI.30, RPI.34, RPI.39, RPI.6, RPI.9, SV1.1, SV10.1, SV2.3, SV3.3, SV4.3, SV5.3, SV6.3, SV7.3, SV8.3, SV9.3, U$1.ADDR, U$6.GND1, U$6.GND2, U$6.GND3, U$6.GND4, U$6.MISO/CFG_COM1, U$6.VDDUSB; no longer U$1.AGND
- net N$4: now also U$1.AIN0; no longer U$1.CH0
- net RPI10: now also U$6.TXD1
- net RPI19: now also SV1.6; no longer U$1.MOSI
- net RPI2: now also Q1.S, U$2.5
- net RPI21: now also SV1.7; no longer U$1.MISO
- net RPI23: now also SV1.5; no longer U$1.SCK
- net RPI24: now also SV1.4
- net RPI26: no longer U$1.!CS
- net RPI3: now also U$1.SDA
- net RPI5: now also U$1.SCL
- net RPI8: now also U$6.RXD1
